Commit message: Autonomous Navigation Robot - VSLAM

File: description/depth_camera.xacro (robot description, xacro)
@@ -21,26 +21,21 @@
     <link name="camera_link_optical"></link>
     <gazebo reference="camera_link">
-        <material>Gazebo/Red</material>
-        <sensor name="camera" type="depth">
-            <pose> 0 0 0 0 0 0 </pose>
-            <visualize>true</visualize>
-            <update_rate>10</update_rate>
+        <sensor name="depth_camera" type="rgbd_camera">
+        <gz_frame_id>camera_link_optical</gz_frame_id>
+            <always_on>true</always_on>
+            <update_rate>5</update_rate>
+            <topic>depth_camera</topic>
             <camera>
                 <horizontal_fov>1.089</horizontal_fov>
                 <image>
-                    <format>B8G8R8</format>
                     <width>640</width>
                     <height>480</height>
+                    <format>R8G8B8</format>
                 </image>
                 <clip>
                     <near>0.05</near>
-                    <far>8.0</far>
+                    <far>15.0</far>
                 </clip>
             </camera>
-            <plugin name="camera_controller" filename="libgazebo_ros_camera.so">
-                <frame_name>camera_link_optical</frame_name>
-                <min_depth>0.1</min_depth>
-                <max_depth>100.0</max_depth>
-            </plugin>
         </sensor>
     </gazebo>

File: description/ros2_control.xacro (robot description, xacro)
@@ -4,5 +4,5 @@
         <ros2_control name="RealRobot" type="system">
             <hardware>
-                <plugin>diffdrive_arduino/DiffDriveArduinoHardware</plugin>
+                <plugin>gz_ros2_control/GazeboSimSystem</plugin>
                 <param name="left_wheel_name">left_wheel_joint</param>
                 <param name="right_wheel_name">right_wheel_joint</param>
@@ -55,7 +55,6 @@
     </xacro:if>
     <gazebo>
-        <plugin name="gz_ros2_control::GazeboSimROS2ControlPlugin" filename="libgz_ros2_control-system.so">
+        <plugin filename="gz_ros2_control-system" name="gz_ros2_control::GazeboSimROS2ControlPlugin">
             <parameters>$(find articubot_one)/config/my_controllers.yaml</parameters>
-            <parameters>$(find articubot_one)/config/gaz_ros2_ctl_use_sim.yaml</parameters>
         </plugin>
     </gazebo>
